File: Cashout Station KiCAD Files/Cashout Station.kicad_sch (KiCad schematic)
At the start: 1 part

Commit message: Created PCB
Parts:
- added BT1: Battery_Cell, Connector_PinHeader_2.54mm:PinHeader_1x02_P2.54mm_Vertical, symbol Device:Battery_Cell
- added C1, C2: 100 µF, Capacitor_THT:CP_Radial_D5.0mm_P2.50mm, symbol Device:C_Polarized
- added D1, D2: LED, LED_THT:LED_D5.0mm, symbol Device:LED
- added J1: Adafruit Industries LLC 3885, Connector_PinHeader_2.54mm:PinHeader_1x03_P2.54mm_Vertical, symbol Connector:Conn_01x03_Pin
- added M1, M2: Motor_Servo, Connector_PinHeader_2.54mm:PinHeader_1x03_P2.54mm_Vertical, symbol Motor:Motor_Servo
- added R1, R4: 220Ω, Resistor_THT:R_Axial_DIN0207_L6.3mm_D2.5mm_P7.62mm_Horizontal, symbol Device:R
- added R2, R3: 4.7kΩ, Resistor_THT:R_Axial_DIN0207_L6.3mm_D2.5mm_P7.62mm_Horizontal, symbol Device:R
- added SW1, SW2: SW_Push, Button_Switch_THT:SW_PUSH_6mm, symbol Switch:SW_Push
- added U1: XIAO-ESP32-C6, Library:XIAO-Generic-Thruhole-14P-2.54-21X17.8MM, symbol Seeed_Studio_XIAO_Series(1):XIAO_ESP32-C6-DIP
- added U2: XL1509-5.0, Connector_PinHeader_2.54mm:PinHeader_1x04_P2.54mm_Vertical, symbol Regulator_Switching:XL1509-5.0
- NFC_Connect1: footprint (none) -> Connector_PinHeader_2.54mm:PinHeader_1x04_P2.54mm_Vertical
Connections:
- net at NFC_Connect1.1 (SCL): now also R2.2
- net at NFC_Connect1.2 (SDA): now also R3.2
- net +3.3V: now reaches NFC_Connect1.3 (VCC)
- net +3.3V: now also U1.12 (3V3)
- net GND: now reaches NFC_Connect1.4 (GND)
- net GND: now also BT1.2 (-), C1.2, C2.2, D1.1 (K), D2.1 (K), J1.1 (Pin_1), M1.3 (-), M2.3 (-), SW1.2, SW2.2, U1.13 (GND), U2.3 (OUT-), U2.4 (VIN-)
- new net: SW1.1, U1.8 (GPIO17/D7/RX)
- new net: M2.1 (PWM), U1.2 (GPIO1/A1/D1)
- new net: D1.2 (A), R1.1
- new net: R1.2, U1.4 (GPIO21/D3)
- new net: BT1.1 (+), U2.1 (VIN+)
- new net: D2.2 (A), R4.1
- new net: M1.1 (PWM), U1.1 (GPIO0/A0/D0)
- new net: R4.2, U1.3 (GPIO2/A2/D2)
- new net: R3.1, U1.5 (GPIO22/D4/SDA)
- new net: R2.1, U1.6 (GPIO23/D5/SCL)
- new net: J1.3 (Pin_3), U1.7 (GPIO16/D6/TX)
- new net: SW2.1, U1.9 (GPIO19/D8/SCK)
- new net +5V: C1.1, C2.1, J1.2 (Pin_2), M1.2 (+), M2.2 (+), U1.14 (VBUS), U2.2 (OUT+)
- no-connect marks 0 -> 2
Other:
- moved on the sheet: NFC_Connect1
